Commit message: fix donghocnghich.py , increase angle limit in limit_joints.yaml, remove PID comment in combine_controller.yaml

File: src/thietkemoi/thanxe_new_description/urdf/complete_visual.xacro (robot description, xacro)
@@ -37,5 +37,5 @@
     <collision>
         <geometry>
-        <mesh filename="file://$(find thanxe_new_description)/meshes/dausac.stl" scale="0.0009 0.0009 0.0009"/>
+        <mesh filename="file://$(find thanxe_new_description)/meshes/dausac.stl" scale="0.00099 0.00099 0.00099"/>
         </geometry>
     </collision>

Commit message: Tunning MPPI controller

File: src/thietkemoi/thanxe_new_description/urdf/complete_visual.xacro (robot description, xacro)
@@ -72,29 +72,77 @@
     </gazebo>
     <!-- LIDAR -->
-    <link name="laser_frame">
-            <visual>
-                <geometry>
-                    <cylinder radius="0.05" length="0.04"/>
-                </geometry>
-                <material name="red"/>
-            </visual>
-            <collision>
-                <geometry>
-                    <cylinder radius="0.05" length="0.04"/>
-                </geometry>
-            </collision>
-            <xacro:inertial_cylinder mass="0.1" length="0.04" radius="0.05">
-                <origin xyz="0 0 0" rpy="0 0 0"/>
-            </xacro:inertial_cylinder>
-        </link>
-    <joint name="laser_joint" type="fixed">
-            <parent link="base_link"/>
-            <child link="laser_frame"/>
-            <origin xyz="0.95 0 0.55" rpy="0 0 0"/>
-        </joint>
-    <gazebo reference="laser_frame">
+    <link name="front_laser_frame">
+        <visual>
+            <geometry>
+                <cylinder radius="0.05" length="0.04"/>
+            </geometry>
+            <material name="red"/>
+        </visual>
+        <collision>
+            <geometry>
+                <cylinder radius="0.05" length="0.04"/>
+            </geometry>
+        </collision>
+        <xacro:inertial_cylinder mass="0.1" length="0.04" radius="0.05">
+            <origin xyz="0 0 0" rpy="0 0 0"/>
+        </xacro:inertial_cylinder>
+    </link>
+    <joint name="front_laser_joint" type="fixed">
+        <parent link="base_link"/>
+        <child link="front_laser_frame"/>
+        <origin xyz="0.92 0 0.55" rpy="0 0 0"/>
+    </joint>
+    <gazebo reference="front_laser_frame">
         <material>Gazebo/Red</material>
-        <pose> 0 0 0 0 0 0 </pose>
-        <sensor type="ray" name="laser">
+        <sensor type="ray" name="front_laser">
+          <pose> 0 0 0 0 0 0 </pose>
+          <update_rate>15</update_rate>
+          <visualize>false</visualize>
+          <ray>
+            <scan>
+                <horizontal>
+                    <samples>360</samples>
+                    <min_angle>-3.14</min_angle>
+                    <max_angle>3.14</max_angle>
+                </horizontal>
+            </scan>
+            <range>
+                <min>0.1</min>
+                <max>40</max>
+            </range>
+          </ray>
+          <plugin name="front_laser_controller" filename="libgazebo_ros_ray_sensor.so">
+            <ros>
+                <argument>~/out:=scan_front</argument> </ros>
+            <output_type>sensor_msgs/LaserScan</output_type>
+            <frame_name>front_laser_frame</frame_name>
+          </plugin>
+        </sensor>
+    </gazebo>
+    <!-- <link name="rear_laser_frame">
+        <visual>
+            <geometry>
+                <cylinder radius="0.05" length="0.04"/>
+            </geometry>
+            <material name="blue"/>
+        </visual>
+        <collision>
+            <geometry>
+                <cylinder radius="0.05" length="0.04"/>
+            </geometry>
+        </collision>
+        <xacro:inertial_cylinder mass="0.1" length="0.04" radius="0.05">
+            <origin xyz="0 0 0" rpy="0 0 0"/>
+        </xacro:inertial_cylinder>
+    </link>
+    <joint name="rear_laser_joint" type="fixed">
+        <parent link="base_link"/>
+        <child link="rear_laser_frame"/>
+        <origin xyz="-0.92 0 0.55" rpy="0 0 ${pi}"/>
+    </joint>
+    <gazebo reference="rear_laser_frame">
+        <material>Gazebo/Blue</material>
+        <sensor type="ray" name="rear_laser">
+          <pose> 0 0 0 0 0 0 </pose>
           <update_rate>15</update_rate>
           <visualize>false</visualize>
@@ -112,12 +160,11 @@
             </range>
           </ray>
-          <plugin name="laser_controller" filename="libgazebo_ros_ray_sensor.so">
+          <plugin name="rear_laser_controller" filename="libgazebo_ros_ray_sensor.so">
             <ros>
-                <argument>~/out:=scan</argument>
-            </ros>
+                <argument>~/out:=scan_rear</argument> </ros>
             <output_type>sensor_msgs/LaserScan</output_type>
-            <frame_name>laser_frame</frame_name>
+            <frame_name>rear_laser_frame</frame_name>
           </plugin>
         </sensor>
-    </gazebo>
+    </gazebo> -->
 </robot>

File: src/thietkemoi/thanxe_new_description/urdf/thanxe_new.xacro (robot description, xacro)
@@ -24,7 +24,8 @@
   </visual>
   <collision>
-    <origin xyz="0 0 0" rpy="0 0 0"/>
-    <geometry>
-      <mesh filename="file://$(find thanxe_new_description)/meshes/base_link.stl" scale="0.001 0.001 0.001"/>
+    <origin xyz="0 0 0.45" rpy="0 0 0"/>
+    <geometry>
+      <!-- <mesh filename="file://$(find thanxe_new_description)/meshes/base_link.stl" scale="0.001 0.001 0.001"/> -->
+      <box size="1.8 0.85 0.15"/>
     </geometry>
   </collision>
